File: PCB_AranaBot/MosfetDrives.kicad_sch (KiCad schematic)
At the start: 0 parts

Commit message: Update 5
Se añadió parcialmente los elementos del esquematico del Mosfet Driver
Parts:
- added C18: 120p, symbol Device:C
- added C19: 6800p, symbol Device:C
- added C20, C21: 2.2u, symbol Device:C
- added C22, C25: 1u, symbol Device:C
- added C23, C24: 2200p, symbol Device:C
- added C26, C27, C28: 0.015u, symbol Device:C
- added R11: 250k, symbol Device:R
- added R12: 16.2k, symbol Device:R
- added R13: 31.6k, symbol Device:R
- added R14: 10k, symbol Device:R
- added R15, R17: 1, symbol Device:R
- added R16: 56, symbol Device:R
- added U2: DRV8302DCAR, DRV8302DCAR:DCA56_6P35X3P61, symbol DRV8302DCAR:DRV8302DCAR
Connections:
- new net: C20.2, U2.13 (GVDD)
- new net: C27.2, C28.2, U2.54 (PVDD2)
- new net: C25.1, U2.27 (AVDD)
- new net: C18.1, R12.1, U2.2 (COMP)
- new net: R13.2, R14.1, U2.3 (VSENSE)
- new net: C22.2, U2.23 (DVDD)
- new net: C26.2, U2.56 (SS_TR)
- new net: R17.2, U2.26 (SO2)
- new net: C21.1, U2.15 (CP2)
- new net: C21.2, U2.14 (CP1)
- new net: R11.1, U2.1 (RT_CLK)
- new net: R16.2, U2.25 (SO1)
- new net: R15.2, U2.7 (DTC)
- new net: C19.1, R12.2
- new net +5V: R13.1
- new net BR_SO1: R16.1
- new net BR_SO2: C23.2, C24.2, R17.1
- new net DC_CAL: U2.12 (DC_CAL)
- new net EN_GATE: U2.16 (EN_GATE)
- new net FAULT: U2.6 (*FAULT)
- new net GAIN: U2.10 (GAIN)
- new net GND: C18.2, C19.2, C20.1, C22.1, C23.1, C24.1, C25.2, C26.1, R11.2, R14.2, R15.1, U2.28 (AGND), U2.57 (EPAD)
- new net HA: U2.17 (INH_A)
- new net HB: U2.19 (INH_B)
- new net HC: U2.21 (INH_C)
- new net LA: U2.18 (INL_A)
- new net LB: U2.20 (INL_B)
- new net LC: U2.22 (INL_C)
- new net M_OC: U2.9 (M_OC)
- new net M_PWM: U2.8 (M_PWM)
- new net OC_ADJ: U2.11 (OC_ADJ)
- new net REF: U2.24 (REF)
- no-connect marks 0 -> 3
Other:
- note added: "MOSFET DRIVER"

Commit message: Update 6
Se añadió completamentamente el esquemático del Driver Mosfet
Parts:
- added C29, C30, C31, C32, C34, C35, C36: 10u, symbol Device:C
- added C33, C37, C38, C39, C40: 0.1u, symbol Device:C
- added C41: 4.7u, symbol Device:C
- added D4: PMEG6020ER, Diode_SMD:Nexperia_CFP3_SOD-123W, symbol Diode:PMEG6020ER
- added D5: BAT60A, Diode_SMD:D_SOD-323, symbol Diode:BAT60A
- added L1: 22u, symbol Device:L
- added R18: 18k, symbol Device:R
- added R19, R20: 3.3k, symbol Device:R
- added R21, R23, R25: 39k, symbol Device:R
- added R22, R24, R26: 2.2k, symbol Device:R
- C27, C28: value 0.015u -> 10u
Connections:
- net +5V: now also D5.1 (K)
- net GND: now also C27.1, C28.1, C29.1, C30.1, C31.1, C32.1, C34.1, C35.1, C36.1, C40.1, C41.2, D4.2 (A), R19.1, R20.1, R22.1, R24.1, R26.1
- net +VDC: now reaches C27.2, C28.2, U2.54 (PVDD2)
- net +VDC: now also U2.29 (PVDD1), U2.53 (PVDD2), C29.2, C30.2, C31.2, C32.2, C40.2, C41.1
- net SP2: now reaches U2.30 (SP2)
- net SN2: now reaches U2.31 (SN2)
- net SP1: now reaches U2.32 (SP1)
- net SN1: now reaches U2.33 (SN1)
- net SL_C: now reaches U2.34 (SL_C)
- net GL_C: now reaches U2.35 (GL_C)
- net SH_C: now reaches U2.36 (SH_C)
- net SH_C: now also C39.1, R25.2
- net GH_C: now reaches U2.37 (GH_C)
- net at U2.38 (BST_C): now also C39.2
- net SL_B: now reaches U2.39 (SL_B)
- net GL_B: now reaches U2.40 (GL_B)
- net SH_B: now reaches U2.41 (SH_B)
- net SH_B: now also C38.1, R23.2
- net GH_B: now reaches U2.42 (GH_B)
- net at U2.43 (BST_B): now also C38.2
- net SL_A: now reaches U2.44 (SL_A)
- net GL_A: now reaches U2.45 (GL_A)
- net SH_A: now reaches U2.46 (SH_A)
- net SH_A: now also C37.1, R21.2
- net GH_A: now reaches U2.47 (GH_A)
- net at U2.48 (BST_A): now also C37.2
- net at U2.49 (BIAS): now also R20.2
- net at U2.50 (PH): now also U2.51 (PH), C33.1, D4.1 (K), L1.1
- net at U2.52 (BST_BK): now also C33.2
- new net: R18.1, R19.2
- new net: C34.2, C35.2, C36.2, D5.2 (A), L1.2, R18.2
- new net SENS1: R21.1, R22.2, R23.1, R24.2, R25.1, R26.2
