File: PCB_AranaBot/CAN.kicad_sch (KiCad schematic)
At the start: 0 parts

Commit message: Update 7
Finalizacion del esquematico
Parts:
- added C53, C54: 60p, symbol Device:C
- added C55: 2.2u, symbol Device:C
- added D11, D12: 1.5SMCxxCA, Diode_SMD:D_SMC, symbol Diode:1.5SMCxxCA
- added J8: Conn_01x04, symbol Connector_Generic:Conn_01x04
- added R44: 120, symbol Device:R
- added R45, R46: 10, symbol Device:R
- added R47: 10k, symbol Device:R
- added TR1: ETC1-1-13, Transformer_SMD:Transformer_MACOM_SM-22, symbol Transformer:ETC1-1-13
- added U3: SN65HVD230, Package_SO:SOIC-8_3.9x4.9mm_P1.27mm, symbol Interface_CAN_LIN:SN65HVD230
Connections:
- new net: R45.2, TR1.1
- new net: R46.2, TR1.2
- new net: TR1.3, U3.6 (CANL)
- new net: TR1.5, U3.7 (CANH)
- new net: R47.2, U3.8 (Rs)
- new net +3.3V: C55.1, U3.3 (VCC)
- new net +5V: J8.1 (Pin_1)
- new net CAN_RX: U3.4 (R)
- new net CAN_TX: U3.1 (D)
- new net C_CAN_N: C54.1, D12.1 (A1), J8.3 (Pin_3), R44.2, R46.1
- new net C_CAN_P: C53.2, D11.2 (A2), J8.2 (Pin_2), R44.1, R45.1
- new net GND: C53.1, C54.2, C55.2, D11.1 (A1), D12.2 (A2), J8.4 (Pin_4), R47.1, TR1.4 (MP), U3.2 (GND)
- no-connect marks 0 -> 1
