File: PCB_AranaBot/Filters.kicad_sch (KiCad schematic)
At the start: 0 parts

Commit message: Update 7
Finalizacion del esquematico
Parts:
- added C56, C58, C60, C62: 4.7n, symbol Device:C
- added C57, C59, C61, C63: 100n, symbol Device:C
- added J9: Conn_01x06, symbol Connector_Generic:Conn_01x06
- added R48, R50, R52, R54: 2.2k, symbol Device:R
- added R49, R51, R53, R55: 10k, symbol Device:R
Connections:
- new net +3.3V: C57.1, C59.1, C61.1, C63.1, R48.1, R50.1, R52.1, R54.1
- new net +5V: J9.1 (Pin_1)
- new net GND: C56.2, C57.2, C58.2, C59.2, C60.2, C61.2, C62.2, C63.2, J9.6 (Pin_6)
- new net HALL_1_IN: C56.1, J9.3 (Pin_3), R48.2, R49.1
- new net HALL_1_OUT: R49.2
- new net HALL_2_IN: C58.1, J9.4 (Pin_4), R50.2, R51.1
- new net HALL_2_OUT: R51.2
- new net HALL_3_IN: C60.1, J9.5 (Pin_5), R52.2, R53.1
- new net HALL_3_OUT: R53.2
- new net TEMP_IN: C62.1, J9.2 (Pin_2), R54.2, R55.1
- new net TEMP_MOTOR: R55.2
Other:
- note added: "FILTRO HALL_1"
- note added: "FILTRO HALL_2"
- note added: "FILTRO HALL_3"
- note added: "FILTRO TEMPERATURA"
- note added: "HALL ENCODER"
