File: PCB_AranaBot/Mechanical.kicad_sch (KiCad schematic)
At the start: 0 parts

Commit message: Update 7
Finalizacion del esquematico
Parts:
- added H1, H2, H3, H4: MountingHole_Pad, symbol Mechanical:MountingHole_Pad
- added R65, R66, R67, R68: 0, symbol Device:R
Connections:
- new net: H1.1, R65.1
- new net: H2.1, R66.1
- new net: H3.1, R67.1
- new net: H4.1, R68.1
- new net GND: R65.2, R66.2, R67.2, R68.2
