File: PCB_AranaBot/Mosfets.kicad_sch (KiCad schematic)
At the start: 0 parts

Commit message: Update 7
Finalizacion del esquematico
Parts:
- added C42, C44, C46, C47, C49, C50: 2.2u, symbol Device:C
- added C43, C45: 1000p, symbol Device:C
- added D6, D7, D8: PMEG6020ER, Diode_SMD:Nexperia_CFP3_SOD-123W, symbol Diode:PMEG6020ER
- added J4, J5, J6: Fase1, symbol Connector_Generic:Conn_01x01
- added Q1, Q2, Q3, Q4, Q5, Q6: SiR696DP, Package_SO:PowerPAK_SO-8_Single, symbol Transistor_FET:SiR696DP
- added R27, R28, R32, R33, R37, R38: 10, symbol Device:R
- added R29, R34: 10m, symbol Device:R
- added R30, R35, R40: 34.8k, symbol Device:R
- added R31, R36, R41: 4.99k, symbol Device:R
Connections:
- new net: Q6.4 (G), R38.2
- new net: Q2.4 (G), R28.2
- new net: Q4.4 (G), R33.2
- new net: Q5.4 (G), R37.2
- new net: Q1.4 (G), R27.2
- new net: Q3.4 (G), R32.2
- new net +VDC: C42.1, C46.1, C49.1, D6.1 (K), D7.1 (K), D8.1 (K), Q1.5 (D), Q3.5 (D), Q5.5 (D)
- new net ASENSE: C44.1, D6.2 (A), R30.1, R31.2
- new net BSENSE: C47.1, D7.2 (A), R35.1, R36.2
- new net CSENSE: C50.1, D8.2 (A), R40.1, R41.2
- new net GH_A: R27.1
- new net GH_B: R32.1, R37.1
- new net GL_A: R28.1
- new net GL_B: R33.1, R38.1
- new net GND: C42.2, C43.2, C44.2, C45.1, C45.2, C46.2, C47.2, C49.2, C50.2, Q4.1 (S), Q4.2 (S), Q4.3 (S), Q6.1 (S), Q6.2 (S), Q6.3 (S), R29.1, R31.1, R34.1, R34.2, R36.1, R41.1
- new net SH_A: J4.1 (Pin_1), Q1.1 (S), Q1.2 (S), Q1.3 (S), Q2.5 (D), R30.2
- new net SH_B: J5.1 (Pin_1), J6.1 (Pin_1), Q3.1 (S), Q3.2 (S), Q3.3 (S), Q4.5 (D), Q5.1 (S), Q5.2 (S), Q5.3 (S), Q6.5 (D), R35.2, R40.2
- new net SL_A: C43.1, Q2.1 (S), Q2.2 (S), Q2.3 (S), R29.2
Other:
- note added: "MOSFET"
