File: PCB_AranaBot/PCB_AranaBot.kicad_sch (KiCad schematic)
At the start: 0 parts

Commit message: Update 2
Se añadió las hojas jerárquicas y el diagrama de bloques
Other:
- added sheet Block Diagram (BlockDiagram.kicad_sch)
- added sheet CAN (CAN.kicad_sch)
- added sheet Filters (Filters.kicad_sch)
- added sheet MCU (MCU.kicad_sch)
- added sheet Mechanical (Mechanical.kicad_sch)
- added sheet Mosfet Drivers (MosfetDrives.kicad_sch)
- added sheet Mosfets (Mosfets.kicad_sch)
- added sheet Overview (Overview.kicad_sch)
- note added: "ArañaBot"

Commit message: Update 7
Finalizacion del esquematico
Other:
- sheet Overview renamed InputProtection
- added sheet StepDown (StepDown.kicad_sch)
- added sheet USB (USB.kicad_sch)
- sheet InputProtection: file Overview.kicad_sch -> InputProtection.kicad_sch
Changed lines of the file:
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@@
+	)
+	(sheet
+		(at 204.47 73.66)
+		(size 25.4 21.59)
+		(fields_autoplaced yes)
+		(stroke
+			(width 0.1524)
+			(type solid)
+		)
+		(fill
+			(color 0 0 0 0.0000)
+		)
+		(property "Sheetname" "StepDown"
+			(at 204.47 72.9484 0)
+			(effects
+				(font
+					(size 1.27 1.27)
+				)
+				(justify left bottom)
+			)
+		)
+		(property "Sheetfile" "StepDown.kicad_sch"
+			(at 204.47 95.8346 0)
+			(effects
+				(font
+					(size 1.27 1.27)
+				)
+				(justify left top)
+			)
+		)
+		(instances
+			(project "PCB_AranaBot"
+				(path "/ab14c721-0523-45ec-9912-f84b74b72c79"
+					(page "11")
+				)
+			)
+		)
+	)
+	(sheet
+		(at 175.26 73.66)
+		(size 25.4 21.59)
+		(fields_autoplaced yes)
+		(stroke
+			(width 0.1524)
+			(type solid)
+		)
+		(fill
+			(color 0 0 0 0.0000)
+		)
+		(property "Sheetname" "USB"
+			(at 175.26 72.9484 0)
+			(effects
+				(font
+					(size 1.27 1.27)
+				)
+				(justify left bottom)
+			)
+		)
+		(property "Sheetfile" "USB.kicad_sch"
+			(at 175.26 95.8346 0)
+			(effects
+				(font
+					(size 1.27 1.27)
+				)
+				(justify left top)
+			)
+		)
+		(instances
+			(project "PCB_AranaBot"
+				(path "/ab14c721-0523-45ec-9912-f84b74b72c79"
+					(page "10")
+				)
+			)
+		)
 	)
 	(sheet
@@
 			(color 0 0 0 0.0000)
 		)
-		(property "Sheetname" "Overview"
+		(property "Sheetname" "InputProtection"
 			(at 19.05 41.1984 0)
 			(effects
@@
 			)
 		)
-		(property "Sheetfile" "Overview.kicad_sch"
+		(property "Sheetfile" "InputProtection.kicad_sch"
 			(at 19.05 64.0846 0)
 			(effects
